File: due_can_shield_v11.brd (EAGLE design)
At the start: 115.2 x 57.3 mm, 73 parts, among them IC1 ILD213T, IC2 ILD213T, J1 MOLEX_20P_MINIFIT, Q1 BSP295, Q2 BSP295, Q3 BSP295, Q4 BSP295, U1 SN65HVD234, U2 SN74AHC1G08, U3 SN74AHC1G08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

Commit message: Add files via upload
Parts:
- turned JP1 to 90 degrees
Routing:
- net 53: track 113.1 -> 82.5 mm, vias 3 -> 1
- net 51: track 103.9 -> 75.9 mm, vias 5 -> 1
- net O1: track 53.2 -> 54.7 mm
- net O4: track 70.2 -> 71.1 mm
